Commit message: fix typo

File: src/franka_ros_ultra/franka_description/robots/panda_arm.urdf (robot description, URDF)
Before this commit: robot panda, 17 links, 16 joints
Links:
- added link panda_transducer; collision mesh filename=package://franka_description/meshes/collision/transducer.stl; visual mesh filename=package://franka_description/meshes/visual/transducer.dae
- added link panda_transducer_sc; collision cylinder length=0.1 radius=0.05; collision cylinder length=0.1 radius=0.07
- added link panda_transducer_tcp
Joints:
- added joint panda_hand_joint: type fixed, parent panda_link8, child panda_transducer, origin xyz=-0.002 -0.002 0.046 rpy=0 0 0
- added joint panda_transducer_sc_joint: type fixed, parent panda_transducer, child panda_transducer_sc, origin rpy=0 0 0
- added joint panda_transducer_tcp_joint: type fixed, parent panda_transducer, child panda_transducer_tcp, origin xyz=0 0 0.1034 rpy=0 0 0

File: src/franka_ros_ultra/franka_description/robots/panda_arm.urdf.xacro (robot description, xacro)
@@ -8,5 +8,5 @@
   <xacro:arg name="gazebo" default="false" />
   <!-- Should a transducer be mounted at the flange? yxj20220714" -->
-  <xacro:arg name="transducer" default="false" />
+  <xacro:arg name="transducer" default="true" />
   <xacro:include filename="utils.xacro" />
   <xacro:include filename="panda_arm.xacro" />
