Commit message: urdf for pybullet

File: src/franka_ros_ultra/franka_description/robots/panda_arm.urdf.xacro (robot description, xacro)
@@ -4,9 +4,9 @@
   <xacro:arg name="arm_id" default="panda" />
   <!-- Should a franka_gripper be mounted at the flange?" -->
-  <xacro:arg name="hand" default="false" />
+  <xacro:arg name="hand" default="true" />
   <!-- Is the robot being simulated in gazebo?" -->
   <xacro:arg name="gazebo" default="false" />
   <!-- Should a transducer be mounted at the flange? yxj20220714" -->
-  <xacro:arg name="transducer" default="true" />
+  <xacro:arg name="transducer" default="false" />
   <xacro:include filename="utils.xacro" />
   <xacro:include filename="panda_arm.xacro" />

File: src/franka_ros_ultra/franka_description/robots/panda_arm_false.urdf (robot description, URDF)
Before this commit: robot panda, 20 links, 19 joints
Links:
- removed link panda_transducer
- removed link panda_transducer_sc
- removed link panda_transducer_tcp
Joints:
- removed joint panda_hand_joint
- removed joint panda_transducer_sc_joint
- removed joint panda_transducer_tcp_joint

File: src/franka_ros_ultra/franka_description/robots/panda_arm_hand.urdf (robot description, URDF)
Before this commit: robot panda, 20 links, 19 joints
Links:
- removed link panda_transducer
- removed link panda_transducer_sc
- removed link panda_transducer_tcp
- added link panda_hand; collision mesh filename=package://franka_description/meshes/collision/hand.stl; visual mesh filename=package://franka_description/meshes/visual/hand.dae
- added link panda_hand_sc; collision cylinder length=0.1 radius=0.05; collision cylinder length=0.1 radius=0.07
- added link panda_hand_tcp
- added link panda_leftfinger; collision box size=17.5e-3 15.2e-3 18.5e-3; collision box size=17.5e-3 7e-3 23.5e-3
- added link panda_rightfinger; collision box size=17.5e-3 15.2e-3 18.5e-3; collision box size=17.5e-3 7e-3 23.5e-3
Joints:
- removed joint panda_transducer_sc_joint
- removed joint panda_transducer_tcp_joint
- added joint panda_finger_joint1: type prismatic, parent panda_hand, child panda_leftfinger, origin xyz=0 0 0.0584 rpy=0 0 0, axis 0 1 0, limit lower=0.0 upper=0.04 effort=100 velocity=0.2
- added joint panda_finger_joint2: type prismatic, parent panda_hand, child panda_rightfinger, origin xyz=0 0 0.0584 rpy=0 0 0, axis 0 -1 0, limit lower=0.0 upper=0.04 effort=100 velocity=0.2, mimic joint=panda_finger_joint1
- added joint panda_hand_sc_joint: type fixed, parent panda_hand, child panda_hand_sc, origin rpy=0 0 0
- added joint panda_hand_tcp_joint: type fixed, parent panda_hand, child panda_hand_tcp, origin xyz=0 0 0.1034 rpy=0 0 0
- joint panda_hand_joint: child panda_transducer -> panda_hand; origin xyz=-0.002 -0.002 0.046 rpy=0 0 0 -> xyz=0 0 0 rpy=0 0 -0.7853981633974483
